File: Diagrama/circuito/circuito.kicad_sch (KiCad schematic)
At the start: 8 parts, among them J1 Screw_Terminal_01x03, J2 Screw_Terminal_01x03, K1 SANYOU_SRD_Form_C, Q1 2N2222

Commit message: Terminar circuito
Parts:
- added R2, R3: R, Resistor_THT:R_Axial_DIN0207_L6.3mm_D2.5mm_P10.16mm_Horizontal, symbol Device:R
- C1: footprint (none) -> Capacitor_THT:CP_Radial_D12.5mm_P5.00mm
- J1, J2: footprint (none) -> TerminalBlock:TerminalBlock_bornier-3_P5.08mm
- Q1: footprint (none) -> Package_TO_SOT_THT:TO-92L_HandSolder
- R1: footprint (none) -> Resistor_THT:R_Axial_DIN0207_L6.3mm_D2.5mm_P10.16mm_Horizontal
Connections:
- net GND: now also J1.1 (Pin_1), R3.1; no longer J1.3 (Pin_3)
- net VDC: now also J1.3 (Pin_3); no longer J1.1 (Pin_1)
- net at Q1.2 (B): now also R2.2, R3.2; no longer J1.2 (Pin_2)
- new net: J1.2 (Pin_2), R2.1
Other:
- moved on the sheet: J1, R1
